Commit message: Fixed

File: simulator/urdfs/iscoin_azz.urdf (robot description, URDF)
Before this commit: robot ur, 14 links, 13 joints
Links:
- link pen_link: geometry collision cylinder length=0.26 radius=0.032; visual cylinder length=0.26 radius=0.032
Joints:
- removed joint tool0-pen
- added joint wrist_3-pen: type fixed, parent wrist_3_link, child pen_link, origin xyz=0 0 0.125 rpy=0 0 0
